File: circuit_cad/contec_orientalmotorBX2_converter/contec_orientalmotorBX2_converter.kicad_pcb (KiCad board)
At the start: 2 copper layers, 72 x 95 mm, 47 parts, among them J1 GND, J2 TO MX2 enc, J3 from FIT DO, J4 To MX2 DCN7, J5 FIT CNT(motor MX2), J6 TO MX2 DI, J7 To ENC, J8 FIT CNT, J9 From FIT DO, U1 TPS5430DDA

Commit message: アートワーク途中まで
Parts:
- J2: footprint 00_RSPro:conn_8971247_3V -> 00_RSPro:conn_8971266_3H
- Vin1: footprint 00_RSPro:conn_8971238_2V -> 00_RSPro:conn_8971262_2H
- moved TP7 156.8 mm to (59.0, 60.5), turned to -90 degrees
- moved D9 142.5 mm to (66.0, 129.8), turned to 180 degrees
- moved D8 142.3 mm to (66.0, 124.7), turned to 180 degrees
- moved D7 142.1 mm to (66.0, 119.6), turned to 180 degrees
- moved D6 142.0 mm to (66.0, 114.5), turned to 180 degrees
- moved D5 141.8 mm to (66.0, 109.4), turned to 180 degrees
- moved D4 141.7 mm to (66.0, 104.2), turned to 180 degrees
- moved D3 141.6 mm to (66.0, 99.2), turned to 180 degrees
- moved TP8 141.1 mm to (77.0, 80.0), turned to -90 degrees
- moved TP5 130.5 mm to (90.0, 76.0)
- moved C1 112.8 mm to (93.0, 79.5), turned to 0 degrees
- moved TP2 109.0 mm to (97.5, 83.0), turned to 90 degrees
- moved R7 108.7 mm to (108.0, 88.6)
- moved D1 106.2 mm to (85.0, 84.5), turned to -90 degrees
- moved U1 103.5 mm to (91.8, 86.6), turned to 90 degrees
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Routing:
- net +24V: track 0.00 -> 173.3 mm, vias 0 -> 6
- net +5V: track 0.00 -> 128.9 mm, vias 0 -> 9
- net Net-(D7-A): track 0.00 -> 28.6 mm, vias 0 -> 1
- net Net-(D8-A): track 0.00 -> 25.8 mm, vias 0 -> 5
- net Net-(D1-K): track 0.00 -> 16.7 mm, vias 0 -> 2
- net Net-(D9-A): track 0.00 -> 15.8 mm, vias 0 -> 2
- net Net-(J7-Pin_4): track 0.00 -> 13.7 mm, vias 0 -> 2
- net Net-(J7-Pin_3): track 0.00 -> 13.4 mm, vias 0 -> 2
- net Net-(J7-Pin_2): track 0.00 -> 13.4 mm, vias 0 -> 2
- net Net-(from_DA_output1-Pin_1): track 0.00 -> 11.0 mm, vias 0 -> 1
- net Net-(J2-Pin_2): track 0.00 -> 9.34 mm, vias 0 -> 1
- net Net-(J6-Pin_5): track 0.00 -> 8.76 mm, vias 0 -> 1
- net Net-(J6-Pin_1): track 0.00 -> 8.45 mm, vias 0 -> 1
- net Net-(U1-EN): track 0.00 -> 8.41 mm, vias 0 -> 2
- net Net-(J2-Pin_1): track 0.00 -> 8.09 mm, vias 0 -> 1
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
Commit message: 配線完了
Parts:
- removed TP8: GND, TestPoint:TestPoint_Pad_D1.0mm
- moved TP6 31.4 mm to (104.0, 109.0)
- moved TP7 8.07 mm to (64.5, 66.4)
- moved TP2 3.34 mm to (99.8, 85.5)
- moved TP9 2.26 mm to (116.8, 115.2)
- moved TP3 1.94 mm to (89.8, 93.8)
- moved TP4 1.03 mm to (118.0, 78.8)
- renumbered GND to EARTH
Connections:
- EARTH pad 1: (no net) -> Earth (x4)
Routing:
- net Earth: track 0.00 -> 310.7 mm
- net Net-(D2-A): track 0.00 -> 84.4 mm, vias 0 -> 6
- net Net-(D3-A): track 0.00 -> 75.1 mm, vias 0 -> 6
- net Net-(from_DA_output1-Pin_2): track 0.00 -> 71.5 mm, vias 0 -> 1
- net Net-(D4-A): track 0.00 -> 66.0 mm, vias 0 -> 4
- net Net-(from_DA_output1-Pin_1): track 11.0 -> 69.8 mm, vias 1 -> 2
- net Net-(D5-A): track 7.89 -> 56.9 mm, vias 1 -> 4
- net Net-(D6-A): track 0.00 -> 48.5 mm, vias 0 -> 4
- net Net-(J2-Pin_1): track 8.09 -> 49.5 mm, vias 1 -> 4
- net Net-(J6-Pin_1): track 8.45 -> 47.4 mm, vias 1 -> 2
- net Net-(J2-Pin_2): track 9.34 -> 48.0 mm, vias 1 -> 2
- net Net-(J6-Pin_3): track 7.39 -> 45.0 mm, vias 1 -> 4
- net Net-(J6-Pin_5): track 8.76 -> 40.8 mm
- net Net-(D1-K): track 16.7 -> 34.0 mm
- net Net-(D7-A): track 28.6 -> 38.2 mm, vias 1 -> 4
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- added copper zone on B.Cu, net GND
- added copper zone on F.Cu, net GND

Commit message: TDK追加
Parts:
- added +5V: conn_8971238_2V, 00_RSPro:conn_8971238_2V, F.Cu at (95.5, 119.0)
- FIT DIN: renamed from J9
- MX2_DI CN7: renamed from J6
- renumbered to_BX2 to BX2_Ain, U1 to DCDC1, from_DA_output1 to FIT_AO, J8 to FIT_CNT, J5 to FIT_CNT(motor), J2 to MX2_ENC, J7 to TO_ENCODER, TP4 to TP, TP6 to TP+24V, TP2 to TP_ENABLE, TP7 to TP_GND
Routing:
- net +5V: track 133.3 -> 141.8 mm, vias 4 -> 3
- net Net-(J2-Pin_2): track 48.0 -> 46.7 mm
- net Net-(D2-A): track 84.4 -> 83.5 mm
- net Net-(J2-Pin_1): track 49.5 -> 49.3 mm, vias 4 -> 3
- net GND: vias 0 -> 49
Other:
- board text added: "+24V"
- board text added: "+5V"
- board text added: "+A"
- board text added: "+Ain"
- board text added: "-A"
- board text added: "-Ain"
- board text added: "0-5Vで速度設定"
- board text added: "2024/2"
- board text added: "A+"
- board text added: "A-"
- board text added: "A相"
- board text added: "B相"
- board text added: "CN7 ch4"
- board text added: "CN7 ch5"
- board text added: "CN7 ch6"
- board text added: "CN7 ch7"
- board text added: "CN7 ch8"
- board text added: "CN7 ch9"
- board text added: "CONTEC(FIT)-OrientalMotorMX2 Connection Board"
- board text added: "DC_IN"
- board text added: "Designed by YOSHIDA Yuji"
- board text added: "EARTH"
- board text added: "FIT"
- board text added: "FIT_DO"
- board text added: "FROM_CN7"
- board text added: "GND"
- board text added: "MX2 エンコーダ出力"
- board text added: "Vin"
- board text added: "Z相"
- board text added: "ch2"
- board text added: "ch2とch4をONで正転,ch3とch4をONで逆転"
- board text added: "ch3"
- board text added: "ch4"
- board text added: "ch5"
- board text added: "ch6"
- board text added: "ch7"
- board text added: "ch8"
- board text added: "ch9"
- board text added: "motor_MX2 CN5"
- board text added: "エンコーダ単体接続用"
- board text added: "コンテックとオリエンタルモータMX2を 接続する変換ボード． 24Vの外部電源接続．内部で5V生成． 5Vを直接入力することも可能"
- board text added: "直接5V接続用"
- board text added: "＋５V"
