File: circuit_cad/電流電圧変換器_絶縁型2線式/電流電圧変換器_絶縁型2線式.kicad_sch (KiCad schematic)
At the start: 9 parts, among them J1 Conn_01x02_Pin, J2 Conn_01x03_Pin, J3 Conn_01x04_Pin, U1 CC3-2412Dx-E

Commit message: 発注データ作成
Parts:
- added J4: Conn_01x02_Pin, 00_RSPro:conn_8971262_2H, symbol Connector:Conn_01x02_Pin
- C1: renamed from C2; footprint (none) -> Capacitor_SMD:C_0805_2012Metric
- C2: renamed from C1; footprint (none) -> Capacitor_SMD:C_1206_3216Metric
- J1: footprint (none) -> 00_RSPro:conn_8971262_2H
- J2: footprint (none) -> 00_RSPro:conn_8971266_3H
- J3: footprint (none) -> 00_RSPro:conn_8971275_4H
- R3: value R -> 500; footprint (none) -> 00_Alpha_Electronics:MB_Series
Connections:
- net +A: now reaches J2.1 (Pin_1), J3.3 (Pin_3), R3.2
- net TRM: now reaches R1.2, R2.1, U1.6 (TRM)
- net GND renamed +Vin
- net +Vin: no longer C1.2, C2.1, U1.2 (RC), U1.3 (-Vin)
- new net -Vin: C1.2, C2.1, J4.1 (Pin_1), J4.2 (Pin_2), U1.2 (RC), U1.3 (-Vin)
Other:
- moved on the sheet: J1
